File: eagle/year-shift-r1.brd (EAGLE design)
At the start: 55.5 x 58.4 mm, 23 parts, among them IC1 74HC595D, IC2 74HC595D

Commit message: updates to the board
Parts:
- removed Q1, Q2: (no value), semicon-smd-ipc:SOT23
- added T1, T2: (no value), transistor:TO92-EBC
- SIG_IN, SIG_OUT: device con-lstb:MA07-1 -> con-lstb:MA05-2
- moved SIG_OUT 3.86 mm to (51.4, 47.0), turned to 270 degrees
- moved SIG_IN 3.81 mm to (3.81, 47.0), turned to 270 degrees
Connections:
- net N$41 renamed CLOCK
- net N$42 renamed LATCH
- removed net N$34: SIG_OUT.1
- new net OUT_E: IC1.13, IC2.13, SIG_IN.7, SIG_OUT.7
- new net RESET: IC2.10, SIG_IN.6, SIG_OUT.6
- net EVEN_ANODE: now also T2.C; no longer Q2.3
- net EVEN_SIG: now also SIG_IN.10, SIG_OUT.10, T2.B; no longer Q2.1, SIG_IN.7, SIG_OUT.7
- net GND: now also SIG_IN.1, SIG_OUT.1; no longer IC1.13, IC2.13, SIG_IN.2, SIG_OUT.2
- net ODD_ANODE: now also T1.C; no longer Q1.3
- net ODD_SIG: now also SIG_IN.9, SIG_OUT.9, T1.B; no longer Q1.1, SIG_IN.6, SIG_OUT.6
- net VCC: now also SIG_IN.2, SIG_OUT.2, T1.E, T2.E; no longer IC2.10, Q1.2, Q2.2, SIG_IN.1
Routing:
- net RESET: track 0.00 -> 187.4 mm, vias 0 -> 3
- net OUT_E: track 0.00 -> 143.5 mm, vias 0 -> 5
- net GND: track 62.3 -> 126.4 mm, vias 3 -> 6
- net ODD_SIG: track 79.1 -> 112.2 mm, vias 2 -> 4
- net N$12: track 30.3 -> 61.8 mm
- net EVEN_SIG: track 74.7 -> 99.6 mm, vias 2 -> 3
- net LATCH: track 69.0 -> 92.4 mm
- net ODD_ANODE: track 55.8 -> 75.4 mm, vias 2 -> 5
- net VCC: track 121.9 -> 102.8 mm, vias 3 -> 2
- net N$25: track 32.8 -> 50.2 mm, vias 0 -> 2
- net N$16: track 32.0 -> 48.9 mm, vias 2 -> 4
- net CLOCK: track 101.5 -> 86.3 mm, vias 0 -> 2
- net N$11: track 28.2 -> 19.7 mm
- net N$3: track 33.5 -> 25.1 mm, vias 2 -> 0
- net N$24: track 22.0 -> 29.5 mm
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- added copper zone on layer 16, net N$34
- added copper zone on layer 1, net N$35
