File: eagle/year-shift-r1.sch (EAGLE design)
At the start: 23 parts, among them IC1 74HC595D, IC2 74HC595D

Commit message: updates to the board
Parts:
- removed Q1, Q2: (no value), semicon-smd-ipc:PNP-TRANSISTOR_SOT23
- added T1, T2: (no value), transistor:BC557B-PNP-TO92-EBC
- SIG_IN, SIG_OUT: device con-lstb:MA07-1 -> con-lstb:MA05-2
Connections:
- net N$41 renamed CLOCK
- net N$42 renamed LATCH
- removed net N$34: SIG_OUT.1
- new net OUT_E: IC1A.G, IC2A.G, SIG_IN.7, SIG_OUT.7
- new net RESET: IC2A.SCL, SIG_IN.6, SIG_OUT.6
- net EVEN_ANODE: now also T2.C; no longer Q2.C
- net EVEN_SIG: now also SIG_IN.10, SIG_OUT.10, T2.B; no longer Q2.B, SIG_IN.7, SIG_OUT.7
- net GND: now also SIG_IN.1, SIG_OUT.1; no longer IC1A.G, IC2A.G, SIG_IN.2, SIG_OUT.2
- net ODD_ANODE: now also T1.C; no longer Q1.C
- net ODD_SIG: now also SIG_IN.9, SIG_OUT.9, T1.B; no longer Q1.B, SIG_IN.6, SIG_OUT.6
- net VCC: now also SIG_IN.2, SIG_OUT.2, T1.E, T2.E; no longer IC2A.SCL, Q1.E, Q2.E, SIG_IN.1
