File: eagle/date-led-r1.brd (EAGLE design)
At the start: 91.1 x 39.4 mm, 5 parts

Commit message: More updates
Routing:
- net N$10: track 52.3 -> 56.0 mm
- net N$14: track 59.1 -> 62.2 mm
- net N$9: track 70.6 -> 72.6 mm
- net N$2: track 74.4 -> 76.2 mm
- net N$25: track 73.7 -> 75.1 mm
- net N$1: track 63.7 -> 65.0 mm
- net N$24: track 97.1 -> 98.3 mm
- net N$21: track 44.8 -> 46.0 mm
- net N$28: track 70.5 -> 71.4 mm
- net N$29: track 31.3 -> 32.2 mm
Other:
- board size 91.1 x 39.4 mm -> 91.1 x 36.8 mm
