File: eagle/date-shift-r1.brd (EAGLE design)
At the start: 93.4 x 58.4 mm, 33 parts, among them IC1 74HC595D, IC2 74HC595D, IC3 74HC595D

Commit message: Updated circuit and testing code
Parts:
- added R25, R26: 10k, rcl:R0805
Connections:
- new net LED_PWR: SIG_IN.8, SIG_OUT.8, T1.E, T2.E
- new net N$53: R26.2, T2.B
- new net N$54: R25.2, T1.B
- net EVEN_SIG: now also R26.1; no longer T2.B
- net ODD_SIG: now also R25.1; no longer T1.B
- net VCC: no longer T1.E, T2.E
Routing:
- net EVEN_SIG: track 186.6 -> 180.4 mm
- net VCC: track 225.6 -> 219.5 mm
Changed lines of the file:
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@@
 <element name="R4" library="rcl" package="R0805" value="220" x="20.47875" y="19.20875" rot="MR90"/>
 <element name="R16" library="rcl" package="R0805" value="220" x="22.70125" y="14.44625" rot="MR90"/>
+<element name="R25" library="rcl" package="R0805" value="10k" x="48.26" y="54.61"/>
+<element name="R26" library="rcl" package="R0805" value="10k" x="58.42" y="55.88"/>
 </elements>
 <signals>
@@
 <contactref element="SIG_IN" pad="2"/>
 <contactref element="SIG_OUT" pad="2"/>
-<contactref element="T1" pad="E"/>
-<contactref element="T2" pad="E"/>
 <contactref element="IC1" pad="16"/>
 <contactref element="IC1" pad="16"/>
@@
 <wire x1="64.008" y1="49.276" x2="63.5" y2="49.784" width="0.254" layer="16"/>
 <wire x1="55.372" y1="32.512" x2="55.1434" y2="32.385" width="0.254" layer="16"/>
-<wire x1="64.008" y1="49.276" x2="64.135" y2="48.895" width="0.254" layer="16"/>
 <wire x1="82.804" y1="17.272" x2="82.804" y2="32.512" width="0.254" layer="16"/>
 <wire x1="83.82" y1="16.256" x2="82.804" y2="17.272" width="0.254" layer="16"/>
@@
 <wire x1="60.96" y1="49.784" x2="61.468" y2="50.292" width="0.254" layer="1"/>
 <wire x1="82.804" y1="32.512" x2="82.4484" y2="32.385" width="0.254" layer="16"/>
-<wire x1="67.056" y1="39.116" x2="65.405" y2="37.465" width="0.254" layer="16"/>
 <wire x1="67.056" y1="39.624" x2="67.056" y2="39.116" width="0.254" layer="16"/>
 <wire x1="68.072" y1="40.64" x2="67.056" y2="39.624" width="0.254" layer="1"/>
 <wire x1="89.408" y1="53.34" x2="90.424" y2="52.324" width="0.254" layer="16"/>
 <wire x1="68.58" y1="53.34" x2="89.408" y2="53.34" width="0.254" layer="16"/>
-<wire x1="64.135" y1="48.895" x2="66.548" y2="51.308" width="0.254" layer="16"/>
 <wire x1="66.548" y1="51.308" x2="68.58" y2="53.34" width="0.254" layer="16"/>
 <wire x1="90.424" y1="52.324" x2="90.805" y2="52.07" width="0.254" layer="16"/>
@@
 <via x="83.82" y="16.256" extent="1-16" drill="0.6096" shape="octagon"/>
 <via x="67.056" y="39.624" extent="1-16" drill="0.6096" shape="octagon"/>
+<wire x1="66.548" y1="51.308" x2="67.564" y2="50.292" width="0" layer="19" extent="1-16"/>
 </signal>
 <signal name="SER_IN">
@@
 <contactref element="SIG_IN" pad="9"/>
 <contactref element="SIG_OUT" pad="9"/>
-<contactref element="T1" pad="B"/>
 <wire x1="60.452" y1="46.228" x2="64.008" y2="46.228" width="0.254" layer="16"/>
 <wire x1="59.436" y1="45.212" x2="60.452" y2="46.228" width="0.254" layer="16"/>
@@
 <wire x1="2.54" y1="25.908" x2="8.128" y2="20.32" width="0.254" layer="1"/>
 <wire x1="2.54" y1="41.91" x2="2.54" y2="25.908" width="0.254" layer="16"/>
-<wire x1="64.008" y1="46.228" x2="64.135" y2="46.355" width="0.254" layer="16"/>
 <wire x1="87.884" y1="32.512" x2="87.884" y2="41.656" width="0.254" layer="16"/>
 <wire x1="83.82" y1="28.448" x2="87.884" y2="32.512" width="0.254" layer="16"/>
@@
 <via x="68.58" y="27.94" extent="1-16" drill="0.6096" shape="octagon"/>
 <via x="56.896" y="45.212" extent="1-16" drill="0.6096" shape="octagon"/>
+<contactref element="R25" pad="1"/>
+<wire x1="47.31" y1="54.61" x2="8.128" y2="20.32" width="0" layer="19" extent="1-1"/>
 </signal>
 <signal name="EVEN_SIG">
 <contactref element="SIG_IN" pad="10"/>
 <contactref element="SIG_OUT" pad="10"/>
-<contactref element="T2" pad="B"/>
-<wire x1="60.96" y1="30.48" x2="65.405" y2="34.925" width="0.254" layer="16"/>
 <wire x1="60.96" y1="26.416" x2="60.96" y2="30.48" width="0.254" layer="16"/>
 <wire x1="60.96" y1="24.892" x2="60.96" y2="26.416" width="0.254" layer="1"/>
@@
 <via x="48.768" y="44.704" extent="1-16" drill="0.6096" shape="octagon"/>
 <via x="53.34" y="44.704" extent="1-16" drill="0.6096" shape="octagon"/>
+<contactref element="R26" pad="1"/>
+<wire x1="57.47" y1="55.88" x2="10.16" y2="16.256" width="0" layer="19" extent="1-1"/>
 </signal>
 <signal name="ODD_ANODE">
@@
 <wire x1="3.556" y1="2.54" x2="3.81" y2="2.54" width="0.254" layer="16"/>
 </signal>
+<signal name="N$53">
+<contactref element="R26" pad="2"/>
+<contactref element="T2" pad="B"/>
+<wire x1="59.37" y1="55.88" x2="65.405" y2="34.925" width="0" layer="19" extent="1-1"/>
+</signal>
+<signal name="N$54">
+<contactref element="T1" pad="B"/>
+<contactref element="R25" pad="2"/>
+<wire x1="49.21" y1="54.61" x2="64.135" y2="46.355" width="0" layer="19" extent="1-1"/>
+</signal>
+<signal name="LED_PWR">
+<contactref element="T1" pad="E"/>
+<contactref element="T2" pad="E"/>
+<contactref element="SIG_OUT" pad="8"/>
+<contactref element="SIG_IN" pad="8"/>
+<wire x1="65.405" y1="37.465" x2="90.805" y2="44.45" width="0" layer="19" extent="1-1"/>
+<wire x1="64.135" y1="48.895" x2="65.405" y2="37.465" width="0" layer="19" extent="1-1"/>
+<wire x1="5.08" y1="44.45" x2="64.135" y2="48.895" width="0" layer="19" extent="1-1"/>
+</signal>
 </signals>

Commit message: More updates
Parts:
- R25, R26: value 10k -> 470
Changed lines of the file:
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@@
 <element name="R4" library="rcl" package="R0805" value="220" x="20.47875" y="19.20875" rot="MR90"/>
 <element name="R16" library="rcl" package="R0805" value="220" x="22.70125" y="14.44625" rot="MR90"/>
-<element name="R25" library="rcl" package="R0805" value="10k" x="48.26" y="54.61"/>
-<element name="R26" library="rcl" package="R0805" value="10k" x="58.42" y="55.88"/>
+<element name="R25" library="rcl" package="R0805" value="470" x="48.26" y="54.61"/>
+<element name="R26" library="rcl" package="R0805" value="470" x="58.42" y="55.88"/>
 </elements>
 <signals>
