File: eagle/day-led-r1.brd (EAGLE design)
At the start: 30.1 x 39.4 mm, 2 parts

Commit message: More updates
Routing:
- net N$6: track 75.8 -> 75.3 mm
Other:
- board size 30.1 x 39.4 mm -> 30.1 x 36.8 mm
Changed lines of the file:
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@@
 <plain>
 <wire x1="0" y1="0" x2="30.15" y2="0" width="0.254" layer="20"/>
-<wire x1="30.15" y1="0" x2="30.15" y2="39.36" width="0.254" layer="20"/>
-<wire x1="30.15" y1="39.36" x2="0" y2="39.36" width="0.254" layer="20"/>
-<wire x1="0" y1="39.36" x2="0" y2="0" width="0.254" layer="20"/>
-<hole x="3.81" y="36.83" drill="3.2"/>
-<hole x="26.67" y="36.83" drill="3.2"/>
-<text x="20.955" y="36.5125" size="1.778" layer="16" rot="MR0">DAY REV1</text>
+<wire x1="30.15" y1="0" x2="30.15" y2="36.82" width="0.254" layer="20"/>
+<wire x1="30.15" y1="36.82" x2="0" y2="36.82" width="0.254" layer="20"/>
+<wire x1="0" y1="36.82" x2="0" y2="0" width="0.254" layer="20"/>
+<hole x="3.81" y="34.29" drill="3.2"/>
+<hole x="26.67" y="34.29" drill="3.2"/>
+<text x="20.955" y="33.9725" size="1.778" layer="16" rot="MR0">DAY REV1</text>
 </plain>
 <attributes>
@@
 <contactref element="LED1" pad="18"/>
 <contactref element="SV1" pad="6"/>
-<wire x1="9.398" y1="33.5788" x2="5.08" y2="29.2608" width="0.254" layer="16"/>
-<wire x1="23.5204" y1="33.5788" x2="9.398" y2="33.5788" width="0.254" layer="16"/>
-<wire x1="27.432" y1="29.6672" x2="23.5204" y2="33.5788" width="0.254" layer="16"/>
+<wire x1="8.763" y1="32.9438" x2="5.08" y2="29.2608" width="0.254" layer="16"/>
+<wire x1="24.1554" y1="32.9438" x2="8.763" y2="32.9438" width="0.254" layer="16"/>
+<wire x1="27.432" y1="29.6672" x2="24.1554" y2="32.9438" width="0.254" layer="16"/>
 <wire x1="27.432" y1="28.1305" x2="27.432" y2="29.6672" width="0.254" layer="16"/>
 <wire x1="25.6032" y1="26.3017" x2="27.432" y2="28.1305" width="0.254" layer="16"/>
@@
 <signal name="N$18">
 <polygon width="0.4064" layer="16">
-<vertex x="0" y="39.37"/>
-<vertex x="30.48" y="39.37"/>
+<vertex x="0" y="36.83"/>
+<vertex x="30.48" y="36.83"/>
 <vertex x="30.48" y="0"/>
 <vertex x="0" y="0"/>
