File: eagle/month-led-r1.brd (EAGLE design)
At the start: 56.8 x 39.4 mm, 3 parts

Commit message: More updates
Routing:
- net N$3: track 60.2 -> 65.0 mm
- net N$9: track 83.4 -> 87.4 mm
- net N$8: track 84.9 -> 88.4 mm
- net N$10: track 40.5 -> 42.4 mm
- net N$6: track 94.0 -> 95.6 mm
- net N$5: track 50.3 -> 51.8 mm
- net N$7: track 132.2 -> 133.5 mm
- net N$14: track 77.4 -> 78.6 mm
- net N$13: track 73.7 -> 74.8 mm
- net N$15: track 44.3 -> 45.1 mm
- net N$19: track 41.8 -> 42.3 mm
- removed copper zone on layer 16, net N$18
Other:
- board size 56.8 x 39.4 mm -> 56.8 x 36.8 mm
