File: eagle/time-shift-r1.brd (EAGLE design)
At the start: 93.4 x 58.4 mm, 30 parts, among them IC2 74HC595D, IC3 74HC595D

Commit message: More updates
Parts:
- added SV3: (no value), con-lstb:MA05-1
- R25, R26: value 10k -> 470
- moved R26 53.8 mm to (7.62, 38.1), flipped to the bottom, turned to 180 degrees
- moved R25 47.7 mm to (5.08, 34.3), flipped to the bottom, turned to 180 degrees
- moved T1 32.6 mm to (42.2, 23.5)
- moved R18 27.4 mm to (26.7, 15.9)
- moved R19 27.4 mm to (31.8, 15.9)
- moved R20 27.4 mm to (36.8, 15.9)
- moved R17 27.4 mm to (21.6, 15.9)
- moved R7 26.7 mm to (29.2, 11.4)
- moved R8 26.7 mm to (34.3, 11.4)
- moved R5 26.7 mm to (19.1, 11.4)
- moved R6 26.7 mm to (24.1, 11.4)
- moved IC3 26.4 mm to (53.3, 32.4)
- moved R24 25.1 mm to (62.2, 15.2)
- moved R21 25.0 mm to (47.0, 15.6)
- moved R22 25.0 mm to (52.1, 15.6)
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Connections:
- new net N$42: SV1.5, SV3.5
- new net N$43: R15.2, SV3.2
- new net N$44: R16.2, SV3.4
- net N$38: now also SV3.1
- net N$39: now also SV3.3
Routing:
- net GND: track 0.00 -> 123.1 mm, vias 0 -> 3
- net VCC: track 0.00 -> 120.1 mm, vias 0 -> 4
- net ODD_SIG: track 0.00 -> 114.7 mm, vias 0 -> 6
- net EVEN_SIG: track 0.00 -> 113.0 mm, vias 0 -> 4
- net LATCH: track 0.00 -> 94.6 mm, vias 0 -> 2
- net LED_PWR: track 0.00 -> 94.6 mm, vias 0 -> 3
- net CLOCK: track 0.00 -> 90.8 mm, vias 0 -> 4
- net N$53: track 0.00 -> 86.6 mm, vias 0 -> 2
- net OUT_E: track 0.00 -> 85.4 mm
- net RESET: track 0.00 -> 77.1 mm, vias 0 -> 4
- net N$25: track 0.00 -> 75.2 mm, vias 0 -> 4
- net N$54: track 0.00 -> 56.0 mm, vias 0 -> 2
- net N$16: track 0.00 -> 51.5 mm, vias 0 -> 2
- net ODD_ANODE: track 0.00 -> 50.7 mm, vias 0 -> 2
- net EVEN_ANODE: track 0.00 -> 47.9 mm, vias 0 -> 2
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- added copper zone on layer 1, net N$45
- removed copper zone on layer 1, net N$35
Other:
- board size 93.4 x 58.4 mm -> 70.5 x 55.9 mm
- board text added: "TIME DRV"
- board text removed: "YEAR DISPLAY DRV"
