File: eagle/display-controller.sch (EAGLE design)
At the start: 8 parts

Commit message: Lots of schematics updates and some initial code
Parts:
- R1: value 440 -> 470
Changed lines of the file:
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@@
 <part name="T1" library="transistor" deviceset="*-NPN-" device="TO92-CBE" technology="BC337-40"/>
 <part name="P+6" library="supply1" deviceset="VCC" device=""/>
-<part name="R1" library="rcl" deviceset="R-EU_" device="0207/2V" value="440"/>
+<part name="R1" library="rcl" deviceset="R-EU_" device="0207/2V" value="470"/>
 </parts>
 <sheets>
