File: eagle/main.brd (EAGLE design)
At the start: 100 x 80 mm, 8 parts

Commit message: new boards and source code
Parts:
- added AUDIO_AMPLIFIER: (no value), con-lsta:FE07
- added C1: 32pF, rcl:C025-024X044
- added D1, D2: 1N4004, diode:DO41-10
- added G1: CR2032V, battery:CR2032V
- added HV, LV: (no value), con-lsta:FE06
- added IC1: PCF8583P, ds1307_pcf8583:DIL08
- added PHOTORESISTOR: (no value), pinhead:1X02
- added Q1: 32.768KHz, crystal:TC26H
- added R1, R2: 10k, resistor:M0805
- added R3: 1k, rcl:M0805
- added RADIO_RESET: (no value), con-lsta:FE10
- added SERIAL: (no value), con-lstb:MA05-1
- added U$2: AS1117M3-3, linear_mod_by_bwa:SOT223
- moved A4567 16.6 mm to (26.7, 43.2)
- moved U$1 16.6 mm to (26.7, 61.0)
- moved I2C$1 8.89 mm to (25.4, 30.5)
- moved I2C$2 6.35 mm to (25.4, 25.4)
- moved I2C$6 3.81 mm to (25.4, 5.08)
- moved I2C$3 3.81 mm to (25.4, 20.3)
- moved I2C$4 1.27 mm to (25.4, 15.2)
- moved I2C$5 1.27 mm to (25.4, 10.2)
Connections:
- new net AUDIO_LEFT: AUDIO_AMPLIFIER.7
- new net AUDIO_RIGHT: AUDIO_AMPLIFIER.5
- new net INPUT_INT: U$1.P$6
- new net N$1: C1.1, IC1.1, Q1.2
- new net N$2: IC1.2, Q1.1
- new net N$3: D1.A, G1.+
- new net N$4: C1.2, D1.C, D2.C, IC1.8
- new net N$5: RADIO_RESET.10
- new net N$6: RADIO_RESET.9
- new net N$8: U$1.P$17
- new net PHOTORESISTOR: PHOTORESISTOR.2, R3.2
- new net RADIO_RESET: RADIO_RESET.3, U$1.P$7
- new net RADIO_SDIO: RADIO_RESET.6
- new net RESET: SERIAL.3, U$1.P$22, U$1.P$3
- new net RTC_INT: IC1.7, R1.1, R2.2, U$1.P$5
- new net RX: SERIAL.5, U$1.P$2
- new net SCL_3.3: LV.1, RADIO_RESET.4
- new net SDA_3.3: LV.6, RADIO_RESET.5
- new net TX: SERIAL.4, U$1.P$1
- new net VCC/2: LV.4, RADIO_RESET.7, U$2.2
- net GND: now also AUDIO_AMPLIFIER.1, AUDIO_AMPLIFIER.6, G1.-, HV.3, IC1.3, IC1.4, LV.3, R2.1, R3.1, RADIO_RESET.8, SERIAL.1, U$1.P$23, U$1.P$4, U$2.1
- net SCL: now also A4567.2, HV.1, IC1.6
- net SDA: now also A4567.1, HV.6, IC1.5
- net VCC: now also AUDIO_AMPLIFIER.2, D2.A, HV.4, PHOTORESISTOR.1, R1.2, SERIAL.2, U$1.P$21, U$2.3

Commit message: Updates big and small
Parts:
- added FN1, FN2, FN3, FN4, TOGGLE1, TOGGLE2, TOGGLE3: (no value), pinhead:1X02
- added KEYPAD: (no value), pinhead:1X08
- added R10, R4, R5, R6, R7, R8, R9: 10k, resistor:M0805
- moved U$2 180.1 mm to (73.0, 69.8), flipped to the bottom, turned to 90 degrees
- moved LV 172.1 mm to (66.0, 68.6), turned to 90 degrees
- moved R3 162.2 mm to (45.1, 48.9), flipped to the bottom, turned to 180 degrees
- moved HV 162.1 mm to (55.9, 68.6), turned to 90 degrees
- moved PHOTORESISTOR 159.7 mm to (44.5, 52.1)
- moved AUDIO_AMPLIFIER 137.4 mm to (68.6, 47.0), turned to 90 degrees
- moved RADIO_RESET 129.5 mm to (52.1, 43.2), turned to 90 degrees
- moved SERIAL 121.8 mm to (6.35, 69.8), turned to 270 degrees
- moved R2 115.1 mm to (71.1, 16.5), flipped to the bottom, turned to 270 degrees
- moved R1 108.5 mm to (71.1, 10.2), flipped to the bottom, turned to 270 degrees
- moved C1 78.0 mm to (48.3, 15.2), turned to 180 degrees
- moved D1 70.1 mm to (49.5, 20.3)
- moved D2 62.9 mm to (42.5, 10.2), turned to 270 degrees
- moved G1 18.8 mm to (27.3, 25.4), turned to 180 degrees
- moved A4567 17.3 mm to (10.2, 38.1)
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Connections:
- removed net N$5: RADIO_RESET.10
- removed net N$6: RADIO_RESET.9
- removed net N$8: U$1.P$17
- new net FN1: FN1.2, R7.2, U$1.P$8
- new net FN2: FN2.2, R8.2, U$1.P$9
- new net FN3: A4567.4, FN3.2, R9.2
- new net FN4: A4567.3, FN4.2, R10.2
- new net KCOL1: KEYPAD.3, U$1.P$12
- new net KCOL2: KEYPAD.1, U$1.P$10
- new net KCOL3: KEYPAD.5, U$1.P$14
- new net KROW1: KEYPAD.2, U$1.P$11
- new net KROW2: KEYPAD.7, U$1.P$16
- new net KROW3: KEYPAD.6, U$1.P$15
- new net KROW4: KEYPAD.4, U$1.P$13
- new net TOGGLE1: R4.2, TOGGLE1.2, U$1.P$20
- new net TOGGLE2: R5.2, TOGGLE2.2, U$1.P$19
- new net TOGGLE3: R6.2, TOGGLE3.2, U$1.P$18
- net AUDIO_LEFT: now also RADIO_RESET.10
- net AUDIO_RIGHT: now also RADIO_RESET.9
- net GND: now also R10.1, R4.1, R5.1, R6.1, R7.1, R8.1, R9.1
- net PHOTORESISTOR: now also U$1.P$17
- net VCC: now also FN1.1, FN2.1, FN3.1, FN4.1, TOGGLE1.1, TOGGLE2.1, TOGGLE3.1
Routing:
- net GND: track 0.00 -> 645.8 mm
- net VCC: track 0.00 -> 326.3 mm
- net SDA: track 0.00 -> 169.8 mm, vias 0 -> 2
- net SCL: track 0.00 -> 166.5 mm
- net RTC_INT: track 0.00 -> 94.6 mm
- net RADIO_RESET: track 0.00 -> 63.6 mm
- net FN4: track 0.00 -> 57.2 mm, vias 0 -> 2
- net SDA_3.3: track 0.00 -> 43.0 mm
- net FN3: track 0.00 -> 40.6 mm, vias 0 -> 2
- net N$4: track 0.00 -> 39.5 mm
- net VCC/2: track 0.00 -> 37.6 mm
- net TOGGLE1: track 0.00 -> 35.6 mm
- net SCL_3.3: track 0.00 -> 35.1 mm, vias 0 -> 2
- net RX: track 0.00 -> 34.3 mm
- net RESET: track 0.00 -> 32.7 mm
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- added copper zone on layer 16, net N$5
Other:
- board size 100 x 80 mm -> 78.4 x 80 mm
- board text added: "CLOCK"
- board text added: "REV1"
- board text added: "TIME CIRCUIT"
