File: eagle/main.sch (EAGLE design)
At the start: 8 parts

Commit message: new boards and source code
Parts:
- added AUDIO_AMPLIFIER: (no value), con-lsta:FE07-1
- added C1: 32pF, rcl:C-EU025-024X044
- added D1, D2: 1N4004, diode:1N4004
- added G1: CR2032V, battery:CR2032V
- added HV, LV: (no value), con-lsta:FE06-1
- added IC1: PCF8583P, ds1307_pcf8583:PCF8583P
- added PHOTORESISTOR: (no value), pinhead:PINHD-1X2
- added Q1: 32.768KHz, crystal:CRYSTALTC26H
- added R1, R2: 10k, resistor:R-EU_M0805
- added R3: 1k, rcl:R-EU_M0805
- added RADIO_RESET: (no value), con-lsta:FE10-1
- added SERIAL: (no value), con-lstb:MA05-1
- added U$2: AS1117M3-3, linear_mod_by_bwa:AS1117M3-3
Connections:
- new net AUDIO_LEFT: AUDIO_AMPLIFIER.7
- new net AUDIO_RIGHT: AUDIO_AMPLIFIER.5
- new net INPUT_INT: U$1.D3~
- new net N$1: C1.1, IC1.OSCI, Q1.2
- new net N$2: IC1.OSCO, Q1.1
- new net N$3: D1.A, G1.+
- new net N$4: C1.2, D1.C, D2.C, IC1.VDD
- new net N$5: RADIO_RESET.10
- new net N$6: RADIO_RESET.9
- new net N$8: U$1.A0
- new net PHOTORESISTOR: PHOTORESISTOR.2, R3.2
- new net RADIO_RESET: RADIO_RESET.3, U$1.D4
- new net RADIO_SDIO: RADIO_RESET.6
- new net RESET: SERIAL.3, U$1.RST
- new net RTC_INT: IC1.!INT, R1.1, R2.2, U$1.D2
- new net RX: SERIAL.5, U$1.RXI
- new net SCL_3.3: LV.1, RADIO_RESET.4
- new net SDA_3.3: LV.6, RADIO_RESET.5
- new net TX: SERIAL.4, U$1.TXO
- new net VCC/2: LV.4, RADIO_RESET.7, U$2.VO
- net GND: now also AUDIO_AMPLIFIER.1, AUDIO_AMPLIFIER.6, G1.-, HV.3, IC1.A0, IC1.VSS, LV.3, R2.1, R3.1, RADIO_RESET.8, SERIAL.1, U$1.GND, U$2.GND
- net SCL: now also A4567.2, HV.1, IC1.SCL
- net SDA: now also A4567.1, HV.6, IC1.SDA
- net VCC: now also AUDIO_AMPLIFIER.2, D2.A, HV.4, PHOTORESISTOR.1, R1.2, SERIAL.2, U$1.VCC, U$2.VI

Commit message: Updates big and small
Parts:
- added FN1, FN2, FN3, FN4, TOGGLE1, TOGGLE2, TOGGLE3: (no value), pinhead:PINHD-1X2
- added KEYPAD: (no value), pinhead:PINHD-1X8
- added R10, R4, R5, R6, R7, R8, R9: 10k, resistor:R-EU_M0805
Connections:
- removed net N$5: RADIO_RESET.10
- removed net N$6: RADIO_RESET.9
- removed net N$8: U$1.A0
- new net FN1: FN1.2, R7.2, U$1.D5~
- new net FN2: FN2.2, R8.2, U$1.D6~
- new net FN3: A4567.4, FN3.2, R9.2
- new net FN4: A4567.3, FN4.2, R10.2
- new net KCOL1: KEYPAD.3, U$1.D9~
- new net KCOL2: KEYPAD.1, U$1.D7
- new net KCOL3: KEYPAD.5, U$1.D11~
- new net KROW1: KEYPAD.2, U$1.D8
- new net KROW2: KEYPAD.7, U$1.D13
- new net KROW3: KEYPAD.6, U$1.D12
- new net KROW4: KEYPAD.4, U$1.D10~
- new net TOGGLE1: R4.2, TOGGLE1.2, U$1.A3
- new net TOGGLE2: R5.2, TOGGLE2.2, U$1.A2
- new net TOGGLE3: R6.2, TOGGLE3.2, U$1.A1
- net AUDIO_LEFT: now also RADIO_RESET.10
- net AUDIO_RIGHT: now also RADIO_RESET.9
- net GND: now also R10.1, R4.1, R5.1, R6.1, R7.1, R8.1, R9.1
- net PHOTORESISTOR: now also U$1.A0
- net VCC: now also FN1.1, FN2.1, FN3.1, FN4.1, TOGGLE1.1, TOGGLE2.1, TOGGLE3.1
Other:
- moved on the sheet: HV, LV
