File: eagle/temperature-shift-r1.sch (EAGLE design)
At the start: 29 parts, among them IC2 74HC595N, IC3 74HC595N

Commit message: Updates big and small
Connections:
- net RESET: now also IC2A.SCL
Other:
- moved on the sheet: IC2, IC3
